Commit message: robot_description

File: robot_description/urdf/panda.xacro (robot description, xacro)
@@ -12,4 +12,6 @@
         </xacro:include>
     </xacro:if>
-    <xacro:include filename="$(find robot_description)/urdf/panda_hw_interface.xacro" />
+    <xacro:include filename="$(find robot_description)/urdf/panda_hw_interface.xacro">
+        <xacro:arg name="end_effector" value="$(arg end_effector)" />
+    </xacro:include>
 </robot>

File: robot_description/urdf/panda_hw_interface.xacro (robot description, xacro)
@@ -1,4 +1,5 @@
 <?xml version="1.0"?>
 <robot name="panda" xmlns:xacro="http://www.ros.org/wiki/xacro">
+    <xacro:arg name="end_effector" default="true" />
     <ros2_control name="panda_hw_interface" type="system">
       <hardware>
@@ -126,4 +127,16 @@
         <state_interface name="effort"/>
       </joint>
+      <xacro:if value="$(arg end_effector)">
+        <joint name="panda_finger_joint1">
+          <state_interface name="position"/>
+          <state_interface name="velocity"/>
+          <state_interface name="effort"/>
+        </joint>
+        <joint name="panda_finger_joint2">
+          <state_interface name="position"/>
+          <state_interface name="velocity"/>
+          <state_interface name="effort"/>
+        </joint>
+      </xacro:if>
     </ros2_control>
 </robot>
